File: hardware/RubberDuckyUSB.kicad_pcb (KiCad board)
At the start: 2 copper layers, 56.4 x 62.6 mm, 8 parts, among them J1 USB_A, J4 Conn_02x03_Odd_Even, J5 Conn_01x04_Pin, U1 ATTINY85-20SU

Commit message: Revising hardware files
Parts:
- removed R1, R2: R, Resistor_SMD:R_0805_2012Metric_Pad1.20x1.40mm_HandSolder
Connections:
- R3 pad 1: D- -> Connector-D-
- U1 pad 2: D- -> Connector-D-
- U1 pad 3: D+ -> Connector-D+
Routing:
- net Connector-D+: track 15.2 -> 35.3 mm, vias 0 -> 2
- net D+: track 18.0 -> 0.00 mm, vias 2 -> 0
- net D-: track 16.6 -> 0.00 mm, vias 2 -> 0
- net Connector-D-: track 17.3 -> 33.7 mm, vias 0 -> 2
